Commit message: urdf change
change of the urdf with the one that includes the plastic elements at the bottom of the robot

File: Ros2RhinoUnity/Assets/URDF/my_robot.urdf (robot description, URDF)
Before this commit: robot my_robot, 5 links, 4 joints
Links:
- link base_link: geometry collision mesh filename=package://robot_definition/meshes/bodyD.stl scale=1 1 1; visual mesh filename=package://robot_definition/meshes/bodyD.stl scale=1 1 1
- link left_wheel: geometry collision mesh filename=package://robot_definition/meshes/leftwheelE.stl scale=1 1 1; visual mesh filename=package://robot_definition/meshes/leftwheelE.stl scale=1 1 1
- link right_wheel: geometry collision mesh filename=package://robot_definition/meshes/rightwheelE.stl scale=1 1 1; visual mesh filename=package://robot_definition/meshes/rightwheelE.stl scale=1 1 1

Commit message: new urdf
wheels are better, still colliding with the floor

File: Ros2RhinoUnity/Assets/URDF/my_robot.urdf (robot description, URDF)
Before this commit: robot my_robot, 5 links, 4 joints
Links:
- link base_link: geometry collision mesh filename=package://robot_definition/meshes/nbody4Nf.stl scale=1 1 1; visual mesh filename=package://robot_definition/meshes/nbody4Nf.stl scale=1 1 1

Commit message: caster wheel try. high friction issue

File: Ros2RhinoUnity/Assets/URDF/my_robot.urdf (robot description, URDF)
Before this commit: robot my_robot, 5 links, 4 joints
Links:
- added link caster_wheel_back, mass 0.00086; collision sphere radius=0.006; visual sphere radius=0.006
- added link caster_wheel_front, mass 0.00086; collision sphere radius=0.006; visual sphere radius=0.006
- link base_link: geometry collision mesh filename=package://robot_definition/meshes/bodyF.stl scale=1 1 1; visual mesh filename=package://robot_definition/meshes/bodyF.stl scale=1 1 1
Joints:
- added joint back_caster_joint: type continuous, parent base_link, child caster_wheel_back, origin xyz=0 -0.051640 -0.040125 rpy=0 0 0, axis -1 0 0
- added joint front_caster_joint: type continuous, parent base_link, child caster_wheel_front, origin xyz=0 0.044373 -0.040125 rpy=0 0 0, axis -1 0 0
